File: Project-6-Full-Integration-Capstone/kicad-project/Integration-Capstone-Board.kicad_pcb (KiCad board)
At the start: 2 copper layers, 65.4 x 39 mm, 42 parts, among them J1 Conn_01x02, J2 Conn_01x02, J3 Conn_01x02, J4 Conn_01x04, J5 Conn_01x07, J6 Conn_01x04, J7 Conn_01x12, J8 Conn_01x04, J9 USB_B_Micro, SW1 SW_SPST, U1 AMS1117-3.3, U2 STM32F411RETx, U3 USBLC6-2SC6, Y1 Crystal

Commit message: Integration-Capstone-Board-Update
Connections:
- U2 pad 33: I2C2_SDA -> unconnected-(U2-PB12-Pad33)
- U2 pad 62: unconnected-(U2-PB9-Pad62) -> I2C2_SDA
Routing:
- net I2C2_SDA: track 32.1 -> 81.4 mm, vias 1 -> 4
Other:
- board size 65.4 x 39 mm -> 65.4 x 39.6 mm
Changed lines of the file:
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@@
 	(net 30 "USB_D-")
 	(net 31 "LED_GESTURE")
-	(net 32 "unconnected-(U2-PB9-Pad62)")
+	(net 32 "unconnected-(U2-PB12-Pad33)")
 	(net 33 "unconnected-(U2-PA14-Pad49)")
 	(net 34 "unconnected-(U2-PB2-Pad28)")
@@
 		(tags "capacitor")
 		(property "Reference" "C12"
-			(at 2.12 0.03 90)
+			(at -1.05 -1 90)
 			(layer "F.SilkS")
 			(effects
@@
 			(layers "F.Cu" "F.Mask" "F.Paste")
 			(roundrect_rratio 0.25)
-			(net 19 "I2C2_SDA")
+			(net 32 "unconnected-(U2-PB12-Pad33)")
 			(pinfunction "PB12")
-			(pintype "bidirectional")
+			(pintype "bidirectional+no_connect")
 		)
 		(pad "34" smd roundrect
@@
 			(layers "F.Cu" "F.Mask" "F.Paste")
 			(roundrect_rratio 0.25)
-			(net 32 "unconnected-(U2-PB9-Pad62)")
+			(net 19 "I2C2_SDA")
 			(pinfunction "PB9")
-			(pintype "bidirectional+no_connect")
+			(pintype "bidirectional")
 		)
 		(pad "63" smd roundrect
@@
 	)
 	(gr_rect
-		(start 90.9 48.6)
+		(start 90.9 48)
 		(end 156.3 87.6)
 		(stroke
@@
 	)
 	(segment
-		(start 139.625 58.458884)
-		(end 139.625 58.175)
-		(width 0.25)
-		(layer "B.Cu")
-		(net 17)
-	)
-	(segment
-		(start 136.433884 61.625)
-		(end 136.8 61.258884)
-		(width 0.25)
-		(layer "B.Cu")
-		(net 17)
-	)
-	(segment
-		(start 136.433884 61.85)
-		(end 136.433884 61.625)
+		(start 140.4 55.14)
+		(end 136.86 51.6)
 		(width 0.25)
 		(layer "B.Cu")
@@
 	)
 	(segment
-		(start 140.4 57.4)
+		(start 140.4 57.883884)
 		(end 140.4 55.14)
 		(width 0.25)
@@
 	)
 	(segment
-		(start 136.8 61.213172)
-		(end 139.188172 58.825)
-		(width 0.25)
-		(layer "B.Cu")
-		(net 17)
-	)
-	(segment
-		(start 139.258884 58.825)
-		(end 139.625 58.458884)
-		(width 0.25)
-		(layer "B.Cu")
-		(net 17)
-	)
-	(segment
 		(start 131.995209 66.288675)
-		(end 136.433884 61.85)
-		(width 0.25)
-		(layer "B.Cu")
-		(net 17)
-	)
-	(segment
-		(start 136.8 61.258884)
-		(end 136.8 61.213172)
-		(width 0.25)
-		(layer "B.Cu")
-		(net 17)
-	)
-	(segment
-		(start 139.625 58.175)
-		(end 140.4 57.4)
-		(width 0.25)
-		(layer "B.Cu")
-		(net 17)
-	)
-	(segment
-		(start 140.4 55.14)
-		(end 136.86 51.6)
-		(width 0.25)
-		(layer "B.Cu")
-		(net 17)
-	)
-	(segment
-		(start 139.188172 58.825)
-		(end 139.258884 58.825)
+		(end 140.4 57.883884)
 		(width 0.25)
 		(layer "B.Cu")
@@
 	)
 	(segment
-		(start 129.6 77.6)
-		(end 129.6 76.125)
-		(width 0.25)
+		(start 139.95 67.65)
+		(end 140.4 67.2)
+		(width 0.2)
 		(layer "F.Cu")
 		(net 19)
 	)
 	(segment
-		(start 129.65 74.75)
-		(end 130 74.4)
-		(width 0.25)
+		(start 140.4 67.2)
+		(end 143.4 67.2)
+		(width 0.2)
 		(layer "F.Cu")
 		(net 19)
 	)
 	(segment
-		(start 129.65 76.075)
-		(end 129.65 74.75)
-		(width 0.25)
+		(start 143.4 67.2)
+		(end 144.6 68.4)
+		(width 0.2)
 		(layer "F.Cu")
 		(net 19)
 	)
 	(segment
-		(start 129.6 76.125)
-		(end 129.65 76.075)
-		(width 0.25)
+		(start 144.6 68.4)
+		(end 144.6 72.6)
+		(width 0.2)
+		(layer "F.Cu")
+		(net 19)
+	)
+	(segment
+		(start 139.6 77.6)
+		(end 137.8 79.4)
+		(width 0.2)
+		(layer "F.Cu")
+		(net 19)
+	)
+	(segment
+		(start 144.6 72.6)
+		(end 144.4 72.8)
+		(width 0.2)
+		(layer "F.Cu")
+		(net 19)
+	)
+	(segment
+		(start 139.075 67.65)
+		(end 139.95 67.65)
+		(width 0.2)
+		(layer "F.Cu")
+		(net 19)
+	)
+	(segment
+		(start 137.8 79.4)
+		(end 136 79.4)
+		(width 0.2)
+		(layer "F.Cu")
+		(net 19)
+	)
+	(segment
+		(start 136 79.4)
+		(end 135.4 78.8)
+		(width 0.2)
 		(layer "F.Cu")
 		(net 19)
 	)
 	(via
-		(at 130 74.4)
+		(at 135.4 78.8)
+		(size 0.6)
+		(drill 0.3)
+		(layers "F.Cu" "B.Cu")
+		(net 19)
+	)
+	(via
+		(at 129.641942 77.641942)
+		(size 0.6)
+		(drill 0.3)
+		(layers "F.Cu" "B.Cu")
+		(net 19)
+	)
+	(via
+		(at 139.6 77.6)
+		(size 0.6)
+		(drill 0.3)
+		(layers "F.Cu" "B.Cu")
+		(net 19)
+	)
+	(via
+		(at 144.4 72.8)
 		(size 0.6)
 		(drill 0.3)
 		(layers "F.Cu" "B.Cu")
-		(free yes)
 		(net 19)
 	)
 	(segment
-		(start 130.73 51.6)
-		(end 123.65 58.68)
-		(width 0.25)
+		(start 135.4 78.8)
+		(end 134.241942 77.641942)
+		(width 0.2)
 		(layer "B.Cu")
 		(net 19)
 	)
 	(segment
-		(start 123.65 66.65)
-		(end 130.4 73.4)
-		(width 0.25)
+		(start 144.4 72.8)
+		(end 139.6 77.6)
+		(width 0.2)
 		(layer "B.Cu")
 		(net 19)
 	)
 	(segment
-		(start 130.4 74)
-		(end 130 74.4)
-		(width 0.25)
+		(start 132.955 49.375)
+		(end 150.28604 49.375)
+		(width 0.2)
 		(layer "B.Cu")
 		(net 19)
 	)
 	(segment
-		(start 130.4 73.4)
-		(end 130.4 74)
-		(width 0.25)
+		(start 148.076346 74.99)
+		(end 146.59 74.99)
+		(width 0.2)
 		(layer "B.Cu")
 		(net 19)
 	)
 	(segment
-		(start 123.65 58.68)
-		(end 123.65 66.65)
-		(width 0.25)
+		(start 150.28604 49.375)
+		(end 151.425 50.51396)
+		(width 0.2)
+		(layer "B.Cu")
+		(net 19)
+	)
+	(segment
+		(start 151.425 50.51396)
+		(end 151.425 71.641346)
+		(width 0.2)
+		(layer "B.Cu")
+		(net 19)
+	)
+	(segment
+		(start 130.73 51.6)
+		(end 132.955 49.375)
+		(width 0.2)
+		(layer "B.Cu")
+		(net 19)
+	)
+	(segment
+		(start 146.59 74.99)
+		(end 144.4 72.8)
+		(width 0.2)
+		(layer "B.Cu")
+		(net 19)
+	)
+	(segment
+		(start 151.425 71.641346)
+		(end 148.076346 74.99)
+		(width 0.2)
+		(layer "B.Cu")
+		(net 19)
+	)
+	(segment
+		(start 134.241942 77.641942)
+		(end 129.641942 77.641942)
+		(width 0.2)
 		(layer "B.Cu")
 		(net 19)
@@
 		(polygon
 			(pts
-				(xy 156.4 48.6) (xy 156.4 87.6) (xy 90.8 87.6) (xy 90.8 48.6)
+				(xy 156.4 48) (xy 156.4 87.6) (xy 90.8 87.6) (xy 90.8 48)
 			)
 		)
